File: outputs.kicad_sch (KiCad schematic)
At the start: 0 parts

Commit message: Schematic done (for now), WIP on layout
Parts:
- added Q10, Q11, Q12, Q9: IRLML6344TRPBF, Package_TO_SOT_SMD:SOT-23_Handsoldering, symbol Transistor_FET:IRLML2060
- added R36, R38, R39, R40, R41, R42, R43: 10k, Resistor_SMD:R_0603_1608Metric_Pad0.98x0.95mm_HandSolder, symbol Device:R
- added R37, R44: 255, Resistor_SMD:R_0603_1608Metric_Pad0.98x0.95mm_HandSolder, symbol Device:R
Connections:
- new net: Q9.3 (D), R37.1
- new net +3V3: Q10.1 (G), R38.2
- new net +5V: R41.2
- new net BUZZER_GND: Q12.3 (D)
- new net BUZZER_ON/OFF: Q12.1 (G), R43.2
- new net GND: Q11.2 (S), Q12.2 (S), Q9.2 (S), R36.1, R40.1, R42.1, R43.1, R44.1
- new net LED_ON_GND: R44.2
- new net LED_RUN: Q9.1 (G), R36.2
- new net LED_RUN_GND: R37.2
- new net SERVO_GND: Q11.3 (D)
- new net SERVO_ON/OFF: Q11.1 (G), R42.2
- new net UART_RX_3V3: R39.1, R40.2
- new net UART_RX_5V: R39.2
- new net UART_TX_3V3: Q10.2 (S), R38.1
- new net UART_TX_5V: Q10.3 (D), R41.1
Other:
- note added: "BUZZER"
- note added: "LED ON"
- note added: "LED RUN"
- note added: "SCREEN"
- note added: "SERVO"
