File: relays.kicad_sch (KiCad schematic)
At the start: 0 parts

Commit message: Schematic done (for now), WIP on layout
Parts:
- added C14, C15, C16: 10uF/16V, Capacitor_SMD:C_0805_2012Metric_Pad1.18x1.45mm_HandSolder, symbol Device:C_Small
- added D6, D7, D8: SBR160S23-7, Diodes_custom:SBR160S23, symbol Device:D
- added Q3, Q4, Q5, Q6, Q7: IRLML6344TRPBF, Package_TO_SOT_SMD:SOT-23_Handsoldering, symbol Transistor_FET:IRLML2060
- added R16, R18, R20, R21, R28, R30: 0, Resistor_SMD:R_0603_1608Metric_Pad0.98x0.95mm_HandSolder, symbol Device:R
- added R17, R19, R29: 4.7k, Resistor_SMD:R_0603_1608Metric_Pad0.98x0.95mm_HandSolder, symbol Device:R
- added R22, R23, R24, R26, R31, R32: 10k, Resistor_SMD:R_0603_1608Metric_Pad0.98x0.95mm_HandSolder, symbol Device:R
- added R25, R27, R33: 255, Resistor_SMD:R_0603_1608Metric_Pad0.98x0.95mm_HandSolder, symbol Device:R
Connections:
- new net +12V: R20.2, R21.2, R30.2
- new net +5V: R16.2, R18.2, R28.2
- new net DEHUM_LED: R33.2
- new net DEHUM_LEVER_F: C16.1, Q6.1 (G), R29.2, R31.2
- new net DEHUM_LEVER_IN: R29.1
- new net DEHUM_RELAY: Q7.1 (G), R32.2
- new net DEHUM_RELAY_+: D8.1 (K), R28.1, R30.1
- new net DEHUM_RELAY_GND: D8.2 (A), Q6.3 (D), Q7.3 (D), R33.1
- new net FAN_LED: R25.2
- new net FAN_LEVER_F: C15.1, R19.2, R23.2
- new net FAN_LEVER_IN: R19.1
- new net FAN_RELAY: Q4.1 (G), R24.2
- new net FAN_RELAY_+: D7.1 (K), R18.1, R21.1
- new net FAN_RELAY_GND: D7.2 (A), Q4.3 (D), R25.1
- new net GND: C14.2, C15.2, C16.2, Q3.2 (S), Q4.2 (S), Q5.2 (S), Q6.2 (S), Q7.2 (S), R22.1, R23.1, R24.1, R26.1, R31.1, R32.1
- new net HEAT_LED: R27.2
- new net HEAT_LEVER_F: C14.1, Q3.1 (G), R17.2, R22.2
- new net HEAT_LEVER_IN: R17.1
- new net HEAT_RELAY: Q5.1 (G), R26.2
- new net HEAT_RELAY_+: D6.1 (K), R16.1, R20.1
- new net HEAT_RELAY_GND: D6.2 (A), Q3.3 (D), Q5.3 (D), R27.1
Other:
- note added: "DEHUM"
- note added: "FAN"
- note added: "HEAT"
