File: ctahr_board.kicad_pcb (KiCad board)
At the start: 2 copper layers, 99 x 70 mm, 104 parts, among them J1 POWER_IN, J10 BUZZER, J11 SERVO, J2 Header_to_RPi, J3 Front panel, J4 DHT INT, J5 DEHUM, J6 FAN, J7 LIGHTSENSOR, J8 DHT EXT, J9 HEAT, Q1 MMBT2369LT1G, Q10 IRLML6344TRPBF, Q11 IRLML6344TRPBF, Q12 IRLML6344TRPBF, Q2 MMBT2369LT1G, Q3 IRLML6344TRPBF, Q4 IRLML6344TRPBF, Q5 IRLML6344TRPBF, Q6 IRLML6344TRPBF, Q7 IRLML6344TRPBF, Q8 MMBT2369LT1G, Q9 IRLML6344TRPBF, U1 L78L33ACUTR, U2 TLC555CDR, U3 TPS54625

Commit message: WIP on layout
Parts:
- C9: moved to B.Cu
- moved J1 256.5 mm to (193.0, 105.0)
- moved F1 243.3 mm to (195.0, 116.5), turned to -90 degrees
- moved D2 230.6 mm to (182.5, 124.5), turned to 180 degrees
- moved D1 223.9 mm to (186.5, 115.1), turned to 90 degrees
- moved C12 213.4 mm to (183.2, 65.5)
- moved C13 213.4 mm to (183.2, 68.0)
- moved D3 208.8 mm to (175.0, 107.5), turned to 180 degrees
- moved D4 199.6 mm to (166.4, 109.0), turned to 90 degrees
- moved R8 198.0 mm to (171.0, 124.5)
- moved R7 195.8 mm to (171.0, 116.0)
- moved R13 192.4 mm to (178.5, 88.6), turned to -90 degrees
- moved R14 187.6 mm to (174.1, 88.8)
- moved R15 187.4 mm to (174.1, 90.5), turned to 180 degrees
- moved C3 140.8 mm to (147.8, 111.5)
- moved C2 132.4 mm to (147.8, 123.5), turned to 180 degrees
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
Commit message: Routing done, need to work on silkscreen
Parts:
- C19, D5, D6, D7, D8, Q10, Q9, R36, R37, R38, R39, R40, R41, R44: moved to B.Cu
- moved Q3 200.9 mm to (171.0, 105.5), turned to -90 degrees
- moved D6 200.8 mm to (172.7, 108.3)
- moved R19 199.9 mm to (194.8, 79.6)
- moved J4 196.0 mm to (178.3, 131.3), turned to 180 degrees
- moved R16 192.9 mm to (174.0, 117.2), turned to -90 degrees
- moved R1 191.6 mm to (174.5, 126.3), turned to 180 degrees
- moved J8 185.8 mm to (166.1, 131.3), turned to 180 degrees
- moved R20 183.2 mm to (170.9, 117.2), turned to -90 degrees
- moved R17 182.4 mm to (171.0, 98.3)
- moved Q4 179.6 mm to (150.2, 105.4), turned to -90 degrees
- moved R2 179.4 mm to (162.1, 126.3), turned to 180 degrees
- moved J11 177.9 mm to (185.6, 112.4), turned to 180 degrees
- moved J3 173.9 mm to (179.8, 83.7)
- moved J10 172.0 mm to (154.1, 131.3), turned to 180 degrees
- moved R18 171.4 mm to (152.7, 117.3), turned to -90 degrees
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Connections:
- net LIGHTSEN_3V3 renamed +3V3
- J2 pad 7: DHT22_EXT -> DHT22_INT
- RV1 pad 1: unconnected-(RV1-Pad1) -> Net-(Q8-C)
- RV1 pad 3: Net-(Q8-C) -> unconnected-(RV1-Pad3)
Routing:
- net +5V: track 0.00 -> 249.7 mm, vias 0 -> 9
- net +12V: track 0.00 -> 202.9 mm, vias 0 -> 4
- net +3V3: track 0.00 -> 198.8 mm, vias 0 -> 1
- net WATCHDOG: track 0.00 -> 149.0 mm, vias 0 -> 1
- net BUZZER_ON/OFF: track 0.00 -> 109.0 mm, vias 0 -> 1
- net POWER_STATE: track 0.00 -> 102.3 mm, vias 0 -> 1
- net VCOND: track 0.00 -> 78.2 mm
- net LIGHT_SENSOR: track 0.00 -> 61.2 mm
- net UART_RX_3V3: track 0.00 -> 59.3 mm, vias 0 -> 2
- net FAN_LEVER_IN: track 0.00 -> 52.6 mm
- net FAN_RELAY: track 0.00 -> 51.1 mm
- net UART_TX_3V3: track 0.00 -> 50.5 mm
- net DEHUM_LEVER_F: track 0.00 -> 42.7 mm
- net DEHUM_RELAY: track 0.00 -> 42.2 mm
- net DHT22_EXT: track 0.00 -> 41.8 mm
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- added copper zone on F.Cu, net +5V
- added copper zone on F.Cu, net Net-(C10-Pad2)
- added copper zone on F.Cu, net VCOND

Commit message: All done, pending review
Parts:
- added U4: ~, Logos:taz, F.Cu at (150.9, 98.3)
- C14, C16, C17, C18, Q11, Q12, Q3, Q4, Q5, Q6, Q7, Q8, R1, R17, R2, R22, R24, R25, R26, R27, R29, R31, R32, R33, R34, R35, R42, R43: moved to B.Cu
- C2, C3: footprint Capacitors:SCMR22J105SRBA0_vertical -> Capacitors:SCMR22G105SRBA0_vertical
- moved RV1 18.6 mm to (114.9, 127.8)
- moved J7 16.6 mm to (128.2, 129.8), turned to 0 degrees
- moved R34 16.0 mm to (129.7, 122.8), turned to 90 degrees
- moved C18 15.6 mm to (124.4, 126.5), turned to -90 degrees
- moved C17 15.5 mm to (126.8, 121.8)
- moved R35 14.1 mm to (127.5, 126.5), turned to -90 degrees
- moved Q8 14.1 mm to (131.1, 126.5)
- moved J10 11.1 mm to (143.2, 129.8), turned to 0 degrees
- moved Q12 9.61 mm to (143.7, 126.4), turned to 180 degrees
- moved J8 8.11 mm to (158.2, 129.8), turned to 0 degrees
- moved D6 6.21 mm to (171.9, 114.5)
- moved R42 6.16 mm to (185.7, 108.0), turned to 90 degrees
- moved D7 5.98 mm to (151.3, 114.5)
- moved D8 5.98 mm to (161.7, 114.5)
- moved J11 5.12 mm to (180.6, 111.3), turned to 0 degrees
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Routing:
- net +3V3: track 198.8 -> 215.5 mm
- net LIGHT_SENSOR: track 61.2 -> 76.6 mm, vias 0 -> 1
- net FAN_RELAY_GND: track 9.22 -> 15.2 mm
- net DEHUM_LEVER_IN: track 19.8 -> 24.0 mm, vias 1 -> 2
- net +12V: track 202.9 -> 199.0 mm, vias 4 -> 5
- net DHT22_INT: track 28.5 -> 24.6 mm
- net HEAT_RELAY_GND: track 15.3 -> 18.8 mm
- net Net-(Q8-C): track 13.4 -> 16.7 mm
- net DEHUM_RELAY_GND: track 15.1 -> 18.3 mm
- net FAN_LEVER_F: track 14.0 -> 17.1 mm
- net BUZZER_GND: track 6.25 -> 3.83 mm
- net FAN_RELAY_+: track 14.4 -> 12.2 mm
- net SERVO_GND: track 5.41 -> 3.25 mm
- net SERVO_ON/OFF: track 20.0 -> 17.9 mm, vias 1 -> 2
- net Net-(C2-Pad2): track 17.0 -> 15.0 mm
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Other:
- board text added: "+12V"
- board text added: "12V"
- board text added: "5V"
- board text added: "CTaHR_board revB https://github.com/Talw3g/ctahr_board"
- board text added: "GND"
- board text added: "POWER IN"
- board text added: "T. MARION - 09/2024"
